File: hack7400/Add.sch (KiCad schematic (older format))
At the start: 4 parts, among them U21 74LS83, U22 74LS83, U23 74LS83, U24 74LS83

Commit message: Updated schematic
Parts:
- U21, U22, U23, U24: footprint (none) -> Package_DIP:DIP-16_W7.62mm_Socket
Changed lines of the file:
@@
 F 0 "U21" H 2100 4181 50  0000 C CNN
 F 1 "74LS83" H 2100 4090 50  0000 C CNN
-F 2 "" H 2100 3200 50  0001 C CNN
+F 2 "Package_DIP:DIP-16_W7.62mm_Socket" H 2100 3200 50  0001 C CNN
 F 3 "http://www.ti.com/lit/gpn/sn74LS83" H 2100 3200 50  0001 C CNN
 	1    2100 3200
@@
 $EndComp
 $Comp
-L power:+5V #PWR?
+L power:+5V #PWR0146
 U 1 1 5F28BDD6
 P 2400 2400
-F 0 "#PWR?" H 2400 2250 50  0001 C CNN
+F 0 "#PWR0146" H 2400 2250 50  0001 C CNN
 F 1 "+5V" H 2415 2573 50  0000 C CNN
 F 2 "" H 2400 2400 50  0001 C CNN
@@
 	2100 2400 2400 2400
 $Comp
-L power:GND #PWR?
+L power:GND #PWR0147
 U 1 1 5F28C95E
 P 2100 4000
-F 0 "#PWR?" H 2100 3750 50  0001 C CNN
+F 0 "#PWR0147" H 2100 3750 50  0001 C CNN
 F 1 "GND" H 2105 3827 50  0000 C CNN
 F 2 "" H 2100 4000 50  0001 C CNN
@@
 F 0 "U22" H 4550 4181 50  0000 C CNN
 F 1 "74LS83" H 4550 4090 50  0000 C CNN
-F 2 "" H 4550 3200 50  0001 C CNN
+F 2 "Package_DIP:DIP-16_W7.62mm_Socket" H 4550 3200 50  0001 C CNN
 F 3 "http://www.ti.com/lit/gpn/sn74LS83" H 4550 3200 50  0001 C CNN
 	1    4550 3200
@@
 $EndComp
 $Comp
-L power:+5V #PWR?
+L power:+5V #PWR0148
 U 1 1 5F28FE5F
 P 4850 2400
-F 0 "#PWR?" H 4850 2250 50  0001 C CNN
+F 0 "#PWR0148" H 4850 2250 50  0001 C CNN
 F 1 "+5V" H 4865 2573 50  0000 C CNN
 F 2 "" H 4850 2400 50  0001 C CNN
@@
 	4550 2400 4850 2400
 $Comp
-L power:GND #PWR?
+L power:GND #PWR0149
 U 1 1 5F28FE6A
 P 4550 4000
-F 0 "#PWR?" H 4550 3750 50  0001 C CNN
+F 0 "#PWR0149" H 4550 3750 50  0001 C CNN
 F 1 "GND" H 4555 3827 50  0000 C CNN
 F 2 "" H 4550 4000 50  0001 C CNN
@@
 F 0 "U23" H 7100 4181 50  0000 C CNN
 F 1 "74LS83" H 7100 4090 50  0000 C CNN
-F 2 "" H 7100 3200 50  0001 C CNN
+F 2 "Package_DIP:DIP-16_W7.62mm_Socket" H 7100 3200 50  0001 C CNN
 F 3 "http://www.ti.com/lit/gpn/sn74LS83" H 7100 3200 50  0001 C CNN
 	1    7100 3200
@@
 $EndComp
 $Comp
-L power:+5V #PWR?
+L power:+5V #PWR0150
 U 1 1 5F2945AD
 P 7400 2400
-F 0 "#PWR?" H 7400 2250 50  0001 C CNN
+F 0 "#PWR0150" H 7400 2250 50  0001 C CNN
 F 1 "+5V" H 7415 2573 50  0000 C CNN
 F 2 "" H 7400 2400 50  0001 C CNN
@@
 	7100 2400 7400 2400
 $Comp
-L power:GND #PWR?
+L power:GND #PWR0151
 U 1 1 5F2945B8
 P 7100 4000
-F 0 "#PWR?" H 7100 3750 50  0001 C CNN
+F 0 "#PWR0151" H 7100 3750 50  0001 C CNN
 F 1 "GND" H 7105 3827 50  0000 C CNN
 F 2 "" H 7100 4000 50  0001 C CNN
@@
 F 0 "U24" H 9550 4181 50  0000 C CNN
 F 1 "74LS83" H 9550 4090 50  0000 C CNN
-F 2 "" H 9550 3200 50  0001 C CNN
+F 2 "Package_DIP:DIP-16_W7.62mm_Socket" H 9550 3200 50  0001 C CNN
 F 3 "http://www.ti.com/lit/gpn/sn74LS83" H 9550 3200 50  0001 C CNN
 	1    9550 3200
@@
 $EndComp
 $Comp
-L power:+5V #PWR?
+L power:+5V #PWR0152
 U 1 1 5F2945D8
 P 9850 2400
-F 0 "#PWR?" H 9850 2250 50  0001 C CNN
+F 0 "#PWR0152" H 9850 2250 50  0001 C CNN
 F 1 "+5V" H 9865 2573 50  0000 C CNN
 F 2 "" H 9850 2400 50  0001 C CNN
@@
 	9550 2400 9850 2400
 $Comp
-L power:GND #PWR?
+L power:GND #PWR0153
 U 1 1 5F2945E3
 P 9550 4000
-F 0 "#PWR?" H 9550 3750 50  0001 C CNN
+F 0 "#PWR0153" H 9550 3750 50  0001 C CNN
 F 1 "GND" H 9555 3827 50  0000 C CNN
 F 2 "" H 9550 4000 50  0001 C CNN
@@
 ADD_OUT_12
 $Comp
-L power:GND #PWR?
+L power:GND #PWR0154
 U 1 1 5F2AA639
 P 1400 2600
-F 0 "#PWR?" H 1400 2350 50  0001 C CNN
+F 0 "#PWR0154" H 1400 2350 50  0001 C CNN
 F 1 "GND" H 1405 2427 50  0000 C CNN
 F 2 "" H 1400 2600 50  0001 C CNN
