File: hack7400/And.sch (KiCad schematic (older format))
At the start: 4 parts, among them U17 74LS08, U18 74LS08, U19 74LS08, U20 74LS08

Commit message: Updated schematic
Parts:
- U17, U18, U19, U20: footprint (none) -> Package_DIP:DIP-14_W7.62mm_Socket
Changed lines of the file:
@@
 F 0 "U17" H 2550 2425 50  0000 C CNN
 F 1 "74LS08" H 2550 2334 50  0000 C CNN
-F 2 "" H 2550 2100 50  0001 C CNN
+F 2 "Package_DIP:DIP-14_W7.62mm_Socket" H 2550 2100 50  0001 C CNN
 F 3 "http://www.ti.com/lit/gpn/sn74LS08" H 2550 2100 50  0001 C CNN
 	1    2550 2100
@@
 F 0 "U17" H 2550 3025 50  0000 C CNN
 F 1 "74LS08" H 2550 2934 50  0000 C CNN
-F 2 "" H 2550 2700 50  0001 C CNN
+F 2 "Package_DIP:DIP-14_W7.62mm_Socket" H 2550 2700 50  0001 C CNN
 F 3 "http://www.ti.com/lit/gpn/sn74LS08" H 2550 2700 50  0001 C CNN
 	2    2550 2700
@@
 F 0 "U17" H 2550 3625 50  0000 C CNN
 F 1 "74LS08" H 2550 3534 50  0000 C CNN
-F 2 "" H 2550 3300 50  0001 C CNN
+F 2 "Package_DIP:DIP-14_W7.62mm_Socket" H 2550 3300 50  0001 C CNN
 F 3 "http://www.ti.com/lit/gpn/sn74LS08" H 2550 3300 50  0001 C CNN
 	3    2550 3300
@@
 F 0 "U17" H 2550 4225 50  0000 C CNN
 F 1 "74LS08" H 2550 4134 50  0000 C CNN
-F 2 "" H 2550 3900 50  0001 C CNN
+F 2 "Package_DIP:DIP-14_W7.62mm_Socket" H 2550 3900 50  0001 C CNN
 F 3 "http://www.ti.com/lit/gpn/sn74LS08" H 2550 3900 50  0001 C CNN
 	4    2550 3900
@@
 F 0 "U17" H 2730 5046 50  0000 L CNN
 F 1 "74LS08" H 2730 4955 50  0000 L CNN
-F 2 "" H 2500 5000 50  0001 C CNN
+F 2 "Package_DIP:DIP-14_W7.62mm_Socket" H 2500 5000 50  0001 C CNN
 F 3 "http://www.ti.com/lit/gpn/sn74LS08" H 2500 5000 50  0001 C CNN
 	5    2500 5000
@@
 AND_OUT_3
 $Comp
-L power:GND #PWR?
+L power:GND #PWR0138
 U 1 1 5F1D73B9
 P 2500 5500
-F 0 "#PWR?" H 2500 5250 50  0001 C CNN
+F 0 "#PWR0138" H 2500 5250 50  0001 C CNN
 F 1 "GND" H 2505 5327 50  0000 C CNN
 F 2 "" H 2500 5500 50  0001 C CNN
@@
 $EndComp
 $Comp
-L power:+5V #PWR?
+L power:+5V #PWR0139
 U 1 1 5F1D7C7C
 P 2500 4500
-F 0 "#PWR?" H 2500 4350 50  0001 C CNN
+F 0 "#PWR0139" H 2500 4350 50  0001 C CNN
 F 1 "+5V" H 2515 4673 50  0000 C CNN
 F 2 "" H 2500 4500 50  0001 C CNN
@@
 F 0 "U18" H 4650 2425 50  0000 C CNN
 F 1 "74LS08" H 4650 2334 50  0000 C CNN
-F 2 "" H 4650 2100 50  0001 C CNN
+F 2 "Package_DIP:DIP-14_W7.62mm_Socket" H 4650 2100 50  0001 C CNN
 F 3 "http://www.ti.com/lit/gpn/sn74LS08" H 4650 2100 50  0001 C CNN
 	1    4650 2100
@@
 F 0 "U18" H 4650 3025 50  0000 C CNN
 F 1 "74LS08" H 4650 2934 50  0000 C CNN
-F 2 "" H 4650 2700 50  0001 C CNN
+F 2 "Package_DIP:DIP-14_W7.62mm_Socket" H 4650 2700 50  0001 C CNN
 F 3 "http://www.ti.com/lit/gpn/sn74LS08" H 4650 2700 50  0001 C CNN
 	2    4650 2700
@@
 F 0 "U18" H 4650 3625 50  0000 C CNN
 F 1 "74LS08" H 4650 3534 50  0000 C CNN
-F 2 "" H 4650 3300 50  0001 C CNN
+F 2 "Package_DIP:DIP-14_W7.62mm_Socket" H 4650 3300 50  0001 C CNN
 F 3 "http://www.ti.com/lit/gpn/sn74LS08" H 4650 3300 50  0001 C CNN
 	3    4650 3300
@@
 F 0 "U18" H 4650 4225 50  0000 C CNN
 F 1 "74LS08" H 4650 4134 50  0000 C CNN
-F 2 "" H 4650 3900 50  0001 C CNN
+F 2 "Package_DIP:DIP-14_W7.62mm_Socket" H 4650 3900 50  0001 C CNN
 F 3 "http://www.ti.com/lit/gpn/sn74LS08" H 4650 3900 50  0001 C CNN
 	4    4650 3900
@@
 F 0 "U18" H 4830 5046 50  0000 L CNN
 F 1 "74LS08" H 4830 4955 50  0000 L CNN
-F 2 "" H 4600 5000 50  0001 C CNN
+F 2 "Package_DIP:DIP-14_W7.62mm_Socket" H 4600 5000 50  0001 C CNN
 F 3 "http://www.ti.com/lit/gpn/sn74LS08" H 4600 5000 50  0001 C CNN
 	5    4600 5000
@@
 AND_OUT_7
 $Comp
-L power:GND #PWR?
+L power:GND #PWR0140
 U 1 1 5F1F709D
 P 4600 5500
-F 0 "#PWR?" H 4600 5250 50  0001 C CNN
+F 0 "#PWR0140" H 4600 5250 50  0001 C CNN
 F 1 "GND" H 4605 5327 50  0000 C CNN
 F 2 "" H 4600 5500 50  0001 C CNN
@@
 $EndComp
 $Comp
-L power:+5V #PWR?
+L power:+5V #PWR0141
 U 1 1 5F1F70A7
 P 4600 4500
-F 0 "#PWR?" H 4600 4350 50  0001 C CNN
+F 0 "#PWR0141" H 4600 4350 50  0001 C CNN
 F 1 "+5V" H 4615 4673 50  0000 C CNN
 F 2 "" H 4600 4500 50  0001 C CNN
@@
 F 0 "U19" H 6800 2425 50  0000 C CNN
 F 1 "74LS08" H 6800 2334 50  0000 C CNN
-F 2 "" H 6800 2100 50  0001 C CNN
+F 2 "Package_DIP:DIP-14_W7.62mm_Socket" H 6800 2100 50  0001 C CNN
 F 3 "http://www.ti.com/lit/gpn/sn74LS08" H 6800 2100 50  0001 C CNN
 	1    6800 2100
@@
 F 0 "U19" H 6800 3025 50  0000 C CNN
 F 1 "74LS08" H 6800 2934 50  0000 C CNN
-F 2 "" H 6800 2700 50  0001 C CNN
+F 2 "Package_DIP:DIP-14_W7.62mm_Socket" H 6800 2700 50  0001 C CNN
 F 3 "http://www.ti.com/lit/gpn/sn74LS08" H 6800 2700 50  0001 C CNN
 	2    6800 2700
@@
 F 0 "U19" H 6800 3625 50  0000 C CNN
 F 1 "74LS08" H 6800 3534 50  0000 C CNN
-F 2 "" H 6800 3300 50  0001 C CNN
+F 2 "Package_DIP:DIP-14_W7.62mm_Socket" H 6800 3300 50  0001 C CNN
 F 3 "http://www.ti.com/lit/gpn/sn74LS08" H 6800 3300 50  0001 C CNN
 	3    6800 3300
@@
 F 0 "U19" H 6800 4225 50  0000 C CNN
 F 1 "74LS08" H 6800 4134 50  0000 C CNN
-F 2 "" H 6800 3900 50  0001 C CNN
+F 2 "Package_DIP:DIP-14_W7.62mm_Socket" H 6800 3900 50  0001 C CNN
 F 3 "http://www.ti.com/lit/gpn/sn74LS08" H 6800 3900 50  0001 C CNN
 	4    6800 3900
@@
 F 0 "U19" H 6980 5046 50  0000 L CNN
 F 1 "74LS08" H 6980 4955 50  0000 L CNN
-F 2 "" H 6750 5000 50  0001 C CNN
+F 2 "Package_DIP:DIP-14_W7.62mm_Socket" H 6750 5000 50  0001 C CNN
 F 3 "http://www.ti.com/lit/gpn/sn74LS08" H 6750 5000 50  0001 C CNN
 	5    6750 5000
@@
 AND_OUT_11
 $Comp
-L power:GND #PWR?
+L power:GND #PWR0142
 U 1 1 5F203683
 P 6750 5500
-F 0 "#PWR?" H 6750 5250 50  0001 C CNN
+F 0 "#PWR0142" H 6750 5250 50  0001 C CNN
 F 1 "GND" H 6755 5327 50  0000 C CNN
 F 2 "" H 6750 5500 50  0001 C CNN
@@
 $EndComp
 $Comp
-L power:+5V #PWR?
+L power:+5V #PWR0143
 U 1 1 5F20368D
 P 6750 4500
-F 0 "#PWR?" H 6750 4350 50  0001 C CNN
+F 0 "#PWR0143" H 6750 4350 50  0001 C CNN
 F 1 "+5V" H 6765 4673 50  0000 C CNN
 F 2 "" H 6750 4500 50  0001 C CNN
@@
 F 0 "U20" H 8900 2425 50  0000 C CNN
 F 1 "74LS08" H 8900 2334 50  0000 C CNN
-F 2 "" H 8900 2100 50  0001 C CNN
+F 2 "Package_DIP:DIP-14_W7.62mm_Socket" H 8900 2100 50  0001 C CNN
 F 3 "http://www.ti.com/lit/gpn/sn74LS08" H 8900 2100 50  0001 C CNN
 	1    8900 2100
@@
 F 0 "U20" H 8900 3025 50  0000 C CNN
 F 1 "74LS08" H 8900 2934 50  0000 C CNN
-F 2 "" H 8900 2700 50  0001 C CNN
+F 2 "Package_DIP:DIP-14_W7.62mm_Socket" H 8900 2700 50  0001 C CNN
 F 3 "http://www.ti.com/lit/gpn/sn74LS08" H 8900 2700 50  0001 C CNN
 	2    8900 2700
@@
 F 0 "U20" H 8900 3625 50  0000 C CNN
 F 1 "74LS08" H 8900 3534 50  0000 C CNN
-F 2 "" H 8900 3300 50  0001 C CNN
+F 2 "Package_DIP:DIP-14_W7.62mm_Socket" H 8900 3300 50  0001 C CNN
 F 3 "http://www.ti.com/lit/gpn/sn74LS08" H 8900 3300 50  0001 C CNN
 	3    8900 3300
@@
 F 0 "U20" H 8900 4225 50  0000 C CNN
 F 1 "74LS08" H 8900 4134 50  0000 C CNN
-F 2 "" H 8900 3900 50  0001 C CNN
+F 2 "Package_DIP:DIP-14_W7.62mm_Socket" H 8900 3900 50  0001 C CNN
 F 3 "http://www.ti.com/lit/gpn/sn74LS08" H 8900 3900 50  0001 C CNN
 	4    8900 3900
@@
 F 0 "U20" H 9080 5046 50  0000 L CNN
 F 1 "74LS08" H 9080 4955 50  0000 L CNN
-F 2 "" H 8850 5000 50  0001 C CNN
+F 2 "Package_DIP:DIP-14_W7.62mm_Socket" H 8850 5000 50  0001 C CNN
 F 3 "http://www.ti.com/lit/gpn/sn74LS08" H 8850 5000 50  0001 C CNN
 	5    8850 5000
@@
 AND_OUT_15
 $Comp
-L power:GND #PWR?
+L power:GND #PWR0144
 U 1 1 5F2036D5
 P 8850 5500
-F 0 "#PWR?" H 8850 5250 50  0001 C CNN
+F 0 "#PWR0144" H 8850 5250 50  0001 C CNN
 F 1 "GND" H 8855 5327 50  0000 C CNN
 F 2 "" H 8850 5500 50  0001 C CNN
@@
 $EndComp
 $Comp
-L power:+5V #PWR?
+L power:+5V #PWR0145
 U 1 1 5F2036DF
 P 8850 4500
-F 0 "#PWR?" H 8850 4350 50  0001 C CNN
+F 0 "#PWR0145" H 8850 4350 50  0001 C CNN
 F 1 "+5V" H 8865 4673 50  0000 C CNN
 F 2 "" H 8850 4500 50  0001 C CNN
