File: hack7400/AndAddMultiplex.sch (KiCad schematic (older format))
At the start: 8 parts, among them U25 74LS157, U26 74LS157, U27 74LS157, U28 74LS157, U29 74LS86, U30 74LS86, U31 74LS86, U32 74LS86

Commit message: Updated schematic
Parts:
- U25, U26, U27, U28: footprint (none) -> Package_DIP:DIP-16_W7.62mm_Socket
- U29, U30, U31, U32: footprint (none) -> Package_DIP:DIP-14_W7.62mm_Socket
