File: hack7400/Sign.sch (KiCad schematic (older format))
At the start: 10 parts, among them U33 74LS32, U34 74LS32, U35 74LS02

Commit message: Updated schematic
Parts:
- U33, U34, U35: footprint (none) -> Package_DIP:DIP-14_W7.62mm_Socket
- U36, U37: renamed from U?; footprint (none) -> Package_DIP:DIP-14_W7.62mm_Socket
Changed lines of the file:
@@
 F 0 "U33" H 2800 3625 50  0000 C CNN
 F 1 "74LS32" H 2800 3534 50  0000 C CNN
-F 2 "" H 2800 3300 50  0001 C CNN
+F 2 "Package_DIP:DIP-14_W7.62mm_Socket" H 2800 3300 50  0001 C CNN
 F 3 "http://www.ti.com/lit/gpn/sn74LS32" H 2800 3300 50  0001 C CNN
 	4    2800 3300
@@
 F 0 "U33" H 2800 2975 50  0000 C CNN
 F 1 "74LS32" H 2800 2884 50  0000 C CNN
-F 2 "" H 2800 2650 50  0001 C CNN
+F 2 "Package_DIP:DIP-14_W7.62mm_Socket" H 2800 2650 50  0001 C CNN
 F 3 "http://www.ti.com/lit/gpn/sn74LS32" H 2800 2650 50  0001 C CNN
 	3    2800 2650
@@
 F 0 "U33" H 2800 2325 50  0000 C CNN
 F 1 "74LS32" H 2800 2234 50  0000 C CNN
-F 2 "" H 2800 2000 50  0001 C CNN
+F 2 "Package_DIP:DIP-14_W7.62mm_Socket" H 2800 2000 50  0001 C CNN
 F 3 "http://www.ti.com/lit/gpn/sn74LS32" H 2800 2000 50  0001 C CNN
 	2    2800 2000
@@
 F 0 "U33" H 2800 1675 50  0000 C CNN
 F 1 "74LS32" H 2800 1584 50  0000 C CNN
-F 2 "" H 2800 1350 50  0001 C CNN
+F 2 "Package_DIP:DIP-14_W7.62mm_Socket" H 2800 1350 50  0001 C CNN
 F 3 "http://www.ti.com/lit/gpn/sn74LS32" H 2800 1350 50  0001 C CNN
 	1    2800 1350
@@
 OUT_7
 $Comp
-L power:+5V #PWR?
+L power:+5V #PWR0171
 U 1 1 5F43260B
 P 8700 2700
-F 0 "#PWR?" H 8700 2550 50  0001 C CNN
+F 0 "#PWR0171" H 8700 2550 50  0001 C CNN
 F 1 "+5V" H 8715 2873 50  0000 C CNN
 F 2 "" H 8700 2700 50  0001 C CNN
@@
 $EndComp
 $Comp
-L power:GND #PWR?
+L power:GND #PWR0172
 U 1 1 5F43310B
 P 8700 3700
-F 0 "#PWR?" H 8700 3450 50  0001 C CNN
+F 0 "#PWR0172" H 8700 3450 50  0001 C CNN
 F 1 "GND" H 8705 3527 50  0000 C CNN
 F 2 "" H 8700 3700 50  0001 C CNN
@@
 F 0 "U34" H 9780 3246 50  0000 L CNN
 F 1 "74LS32" H 9780 3155 50  0000 L CNN
-F 2 "" H 9550 3200 50  0001 C CNN
+F 2 "Package_DIP:DIP-14_W7.62mm_Socket" H 9550 3200 50  0001 C CNN
 F 3 "http://www.ti.com/lit/gpn/sn74LS32" H 9550 3200 50  0001 C CNN
 	5    9550 3200
@@
 F 0 "U34" H 8950 4725 50  0000 C CNN
 F 1 "74LS32" H 8950 4634 50  0000 C CNN
-F 2 "" H 8950 4400 50  0001 C CNN
+F 2 "Package_DIP:DIP-14_W7.62mm_Socket" H 8950 4400 50  0001 C CNN
 F 3 "http://www.ti.com/lit/gpn/sn74LS32" H 8950 4400 50  0001 C CNN
 	4    8950 4400
@@
 F 0 "U34" H 4000 2625 50  0000 C CNN
 F 1 "74LS32" H 4000 2534 50  0000 C CNN
-F 2 "" H 4000 2300 50  0001 C CNN
+F 2 "Package_DIP:DIP-14_W7.62mm_Socket" H 4000 2300 50  0001 C CNN
 F 3 "http://www.ti.com/lit/gpn/sn74LS32" H 4000 2300 50  0001 C CNN
 	3    4000 2300
@@
 F 0 "U34" H 3400 3275 50  0000 C CNN
 F 1 "74LS32" H 3400 3184 50  0000 C CNN
-F 2 "" H 3400 2950 50  0001 C CNN
+F 2 "Package_DIP:DIP-14_W7.62mm_Socket" H 3400 2950 50  0001 C CNN
 F 3 "http://www.ti.com/lit/gpn/sn74LS32" H 3400 2950 50  0001 C CNN
 	2    3400 2950
@@
 F 0 "U34" H 3400 1975 50  0000 C CNN
 F 1 "74LS32" H 3400 1884 50  0000 C CNN
-F 2 "" H 3400 1650 50  0001 C CNN
+F 2 "Package_DIP:DIP-14_W7.62mm_Socket" H 3400 1650 50  0001 C CNN
 F 3 "http://www.ti.com/lit/gpn/sn74LS32" H 3400 1650 50  0001 C CNN
 	1    3400 1650
@@
 $EndComp
 $Comp
-L power:+5V #PWR?
+L power:+5V #PWR0173
 U 1 1 5F43537D
 P 9550 2700
-F 0 "#PWR?" H 9550 2550 50  0001 C CNN
+F 0 "#PWR0173" H 9550 2550 50  0001 C CNN
 F 1 "+5V" H 9565 2873 50  0000 C CNN
 F 2 "" H 9550 2700 50  0001 C CNN
@@
 $EndComp
 $Comp
-L power:GND #PWR?
+L power:GND #PWR0174
 U 1 1 5F435387
 P 9550 3700
-F 0 "#PWR?" H 9550 3450 50  0001 C CNN
+F 0 "#PWR0174" H 9550 3450 50  0001 C CNN
 F 1 "GND" H 9555 3527 50  0000 C CNN
 F 2 "" H 9550 3700 50  0001 C CNN
@@
 F 0 "U33" H 8930 3246 50  0000 L CNN
 F 1 "74LS32" H 8930 3155 50  0000 L CNN
-F 2 "" H 8700 3200 50  0001 C CNN
+F 2 "Package_DIP:DIP-14_W7.62mm_Socket" H 8700 3200 50  0001 C CNN
 F 3 "http://www.ti.com/lit/gpn/sn74LS32" H 8700 3200 50  0001 C CNN
 	5    8700 3200
@@
 ZR
 $Comp
-L 74xx:74LS32 U?
+L 74xx:74LS32 U36
 U 4 1 5F4C767B
 P 2800 6000
-F 0 "U?" H 2800 6325 50  0000 C CNN
+F 0 "U36" H 2800 6325 50  0000 C CNN
 F 1 "74LS32" H 2800 6234 50  0000 C CNN
-F 2 "" H 2800 6000 50  0001 C CNN
+F 2 "Package_DIP:DIP-14_W7.62mm_Socket" H 2800 6000 50  0001 C CNN
 F 3 "http://www.ti.com/lit/gpn/sn74LS32" H 2800 6000 50  0001 C CNN
 	4    2800 6000
@@
 $EndComp
 $Comp
-L 74xx:74LS32 U?
+L 74xx:74LS32 U36
 U 3 1 5F4C7685
 P 2800 5350
-F 0 "U?" H 2800 5675 50  0000 C CNN
+F 0 "U36" H 2800 5675 50  0000 C CNN
 F 1 "74LS32" H 2800 5584 50  0000 C CNN
-F 2 "" H 2800 5350 50  0001 C CNN
+F 2 "Package_DIP:DIP-14_W7.62mm_Socket" H 2800 5350 50  0001 C CNN
 F 3 "http://www.ti.com/lit/gpn/sn74LS32" H 2800 5350 50  0001 C CNN
 	3    2800 5350
@@
 $EndComp
 $Comp
-L 74xx:74LS32 U?
+L 74xx:74LS32 U36
 U 2 1 5F4C768F
 P 2800 4700
-F 0 "U?" H 2800 5025 50  0000 C CNN
+F 0 "U36" H 2800 5025 50  0000 C CNN
 F 1 "74LS32" H 2800 4934 50  0000 C CNN
-F 2 "" H 2800 4700 50  0001 C CNN
+F 2 "Package_DIP:DIP-14_W7.62mm_Socket" H 2800 4700 50  0001 C CNN
 F 3 "http://www.ti.com/lit/gpn/sn74LS32" H 2800 4700 50  0001 C CNN
 	2    2800 4700
@@
 $EndComp
 $Comp
-L 74xx:74LS32 U?
+L 74xx:74LS32 U36
 U 1 1 5F4C7699
 P 2800 4050
-F 0 "U?" H 2800 4375 50  0000 C CNN
+F 0 "U36" H 2800 4375 50  0000 C CNN
 F 1 "74LS32" H 2800 4284 50  0000 C CNN
-F 2 "" H 2800 4050 50  0001 C CNN
+F 2 "Package_DIP:DIP-14_W7.62mm_Socket" H 2800 4050 50  0001 C CNN
 F 3 "http://www.ti.com/lit/gpn/sn74LS32" H 2800 4050 50  0001 C CNN
 	1    2800 4050
@@
 OUT_15
 $Comp
-L 74xx:74LS32 U?
+L 74xx:74LS32 U37
 U 3 1 5F4C76AB
 P 4000 5000
-F 0 "U?" H 4000 5325 50  0000 C CNN
+F 0 "U37" H 4000 5325 50  0000 C CNN
 F 1 "74LS32" H 4000 5234 50  0000 C CNN
-F 2 "" H 4000 5000 50  0001 C CNN
+F 2 "Package_DIP:DIP-14_W7.62mm_Socket" H 4000 5000 50  0001 C CNN
 F 3 "http://www.ti.com/lit/gpn/sn74LS32" H 4000 5000 50  0001 C CNN
 	3    4000 5000
@@
 $EndComp
 $Comp
-L 74xx:74LS32 U?
+L 74xx:74LS32 U37
 U 2 1 5F4C76B5
 P 3400 5650
-F 0 "U?" H 3400 5975 50  0000 C CNN
+F 0 "U37" H 3400 5975 50  0000 C CNN
 F 1 "74LS32" H 3400 5884 50  0000 C CNN
-F 2 "" H 3400 5650 50  0001 C CNN
+F 2 "Package_DIP:DIP-14_W7.62mm_Socket" H 3400 5650 50  0001 C CNN
 F 3 "http://www.ti.com/lit/gpn/sn74LS32" H 3400 5650 50  0001 C CNN
 	2    3400 5650
@@
 $EndComp
 $Comp
-L 74xx:74LS32 U?
+L 74xx:74LS32 U37
 U 1 1 5F4C76BF
 P 3400 4350
-F 0 "U?" H 3400 4675 50  0000 C CNN
+F 0 "U37" H 3400 4675 50  0000 C CNN
 F 1 "74LS32" H 3400 4584 50  0000 C CNN
-F 2 "" H 3400 4350 50  0001 C CNN
+F 2 "Package_DIP:DIP-14_W7.62mm_Socket" H 3400 4350 50  0001 C CNN
 F 3 "http://www.ti.com/lit/gpn/sn74LS32" H 3400 4350 50  0001 C CNN
 	1    3400 4350
@@
 F 0 "U35" H 4600 3925 50  0000 C CNN
 F 1 "74LS02" H 4600 3834 50  0000 C CNN
-F 2 "" H 4600 3600 50  0001 C CNN
+F 2 "Package_DIP:DIP-14_W7.62mm_Socket" H 4600 3600 50  0001 C CNN
 F 3 "http://www.ti.com/lit/gpn/sn74ls02" H 4600 3600 50  0001 C CNN
 	1    4600 3600
@@
 F 0 "U35" H 8950 5375 50  0000 C CNN
 F 1 "74LS02" H 8950 5284 50  0000 C CNN
-F 2 "" H 8950 5050 50  0001 C CNN
+F 2 "Package_DIP:DIP-14_W7.62mm_Socket" H 8950 5050 50  0001 C CNN
 F 3 "http://www.ti.com/lit/gpn/sn74ls02" H 8950 5050 50  0001 C CNN
 	2    8950 5050
@@
 F 0 "U35" H 9700 5375 50  0000 C CNN
 F 1 "74LS02" H 9700 5284 50  0000 C CNN
-F 2 "" H 9700 5050 50  0001 C CNN
+F 2 "Package_DIP:DIP-14_W7.62mm_Socket" H 9700 5050 50  0001 C CNN
 F 3 "http://www.ti.com/lit/gpn/sn74ls02" H 9700 5050 50  0001 C CNN
 	3    9700 5050
@@
 F 0 "U35" H 10450 5375 50  0000 C CNN
 F 1 "74LS02" H 10450 5284 50  0000 C CNN
-F 2 "" H 10450 5050 50  0001 C CNN
+F 2 "Package_DIP:DIP-14_W7.62mm_Socket" H 10450 5050 50  0001 C CNN
 F 3 "http://www.ti.com/lit/gpn/sn74ls02" H 10450 5050 50  0001 C CNN
 	4    10450 5050
@@
 F 0 "U35" H 10630 3246 50  0000 L CNN
 F 1 "74LS02" H 10630 3155 50  0000 L CNN
-F 2 "" H 10400 3200 50  0001 C CNN
+F 2 "Package_DIP:DIP-14_W7.62mm_Socket" H 10400 3200 50  0001 C CNN
 F 3 "http://www.ti.com/lit/gpn/sn74ls02" H 10400 3200 50  0001 C CNN
 	5    10400 3200
@@
 $EndComp
 $Comp
-L power:+5V #PWR?
+L power:+5V #PWR0175
 U 1 1 5F50C1FF
 P 10400 2700
-F 0 "#PWR?" H 10400 2550 50  0001 C CNN
+F 0 "#PWR0175" H 10400 2550 50  0001 C CNN
 F 1 "+5V" H 10415 2873 50  0000 C CNN
 F 2 "" H 10400 2700 50  0001 C CNN
@@
 $EndComp
 $Comp
-L power:GND #PWR?
+L power:GND #PWR0176
 U 1 1 5F50D47F
 P 10400 3700
-F 0 "#PWR?" H 10400 3450 50  0001 C CNN
+F 0 "#PWR0176" H 10400 3450 50  0001 C CNN
 F 1 "GND" H 10405 3527 50  0000 C CNN
 F 2 "" H 10400 3700 50  0001 C CNN
