File: hack7400/XMultiplex.sch (KiCad schematic (older format))
At the start: 8 parts, among them U1 74LS157, U2 74LS157, U3 74LS157, U4 74LS157, U5 74LS86, U6 74LS86, U7 74LS86, U8 74LS86

Commit message: Updated schematic
Parts:
- U1, U2, U3, U4: footprint (none) -> Package_DIP:DIP-16_W7.62mm_Socket
- U5, U6, U7, U8: footprint (none) -> Package_DIP:DIP-14_W7.62mm_Socket
