File: hack7400/YMultiplex.sch (KiCad schematic (older format))
At the start: 8 parts, among them U10 74LS157, U11 74LS157, U12 74LS157, U13 74LS86, U14 74LS86, U15 74LS86, U16 74LS86, U9 74LS157

Commit message: Updated schematic
Parts:
- U10, U11, U12, U9: footprint (none) -> Package_DIP:DIP-16_W7.62mm_Socket
- U13, U14, U15, U16: footprint (none) -> Package_DIP:DIP-14_W7.62mm_Socket
