File: hack7400/hack7400.sch (KiCad schematic (older format))
At the start: 5 parts, among them J1 Conn_01x16_Male, J2 Conn_01x06_Male, J3 Conn_01x16_Male, J4 Conn_01x16_Male, J5 Conn_01x02_Male

Commit message: Updated schematic
Parts:
- added D1, D10, D11, D12, D13, D14, D15, D16, D17, D18, D19, D2, D20, D21, D22, D23, D24, D25, D26, D27, D28, D29, D3, D30, D31, D32, D33, D34, D35, D36, D37, D38, D39, D4, D40, D41, D42, D43, D44, D45, D46, D47, D48, D5, D6, D7, D8, D9: RED, LED_THT:LED_D3.0mm, symbol Device:LED
- added D49, D50, D51, D52, D53, D54: BLUE, LED_THT:LED_D3.0mm, symbol Device:LED
- added D55, D56: GREEN, LED_THT:LED_D3.0mm, symbol Device:LED
- added J6: Barrel_Jack, Connector_BarrelJack:BarrelJack_CUI_PJ-102AH_Horizontal, symbol Connector:Barrel_Jack
- added R1, R10, R11, R12, R13, R14, R15, R16, R17, R18, R19, R2, R20, R21, R22, R23, R24, R25, R26, R27, R28, R29, R3, R30, R31, R32, R33, R34, R35, R36, R37, R38, R39, R4, R40, R41, R42, R43, R44, R45, R46, R47, R48, R5, R55, R56, R6, R7, R8, R9: 330, Resistor_THT:R_Axial_DIN0207_L6.3mm_D2.5mm_P7.62mm_Horizontal, symbol Device:R
- added R49, R50, R51, R52, R53, R54: 160, Resistor_THT:R_Axial_DIN0207_L6.3mm_D2.5mm_P7.62mm_Horizontal, symbol Device:R
- J1, J3, J4: footprint (none) -> Connector_IDC:IDC-Header_2x08_P2.54mm_Vertical
- J2: footprint (none) -> Connector_PinHeader_2.54mm:PinHeader_1x06_P2.54mm_Vertical
- J5: footprint (none) -> Connector_PinHeader_2.54mm:PinHeader_1x02_P2.54mm_Vertical
Connections:
- net F: now also D53.2 (A)
- net NG: now also D56.2 (A)
- net NO: now also D54.2 (A)
- net NX: now also D50.2 (A)
- net NY: now also D52.2 (A)
- net OUT_0: now also D33.2 (A)
- net OUT_1: now also D34.2 (A)
- net OUT_10: now also D43.2 (A)
- net OUT_11: now also D44.2 (A)
- net OUT_12: now also D45.2 (A)
- net OUT_13: now also D46.2 (A)
- net OUT_14: now also D47.2 (A)
- net OUT_15: now also D48.2 (A)
- net OUT_2: now also D35.2 (A)
- net OUT_3: now also D36.2 (A)
- net OUT_4: now also D37.2 (A)
- net OUT_5: now also D38.2 (A)
- net OUT_6: now also D39.2 (A)
- net OUT_7: now also D40.2 (A)
- net OUT_8: now also D41.2 (A)
- net OUT_9: now also D42.2 (A)
- net X_0: now also D1.2 (A)
- net X_1: now also D2.2 (A)
- net X_10: now also D11.2 (A)
- net X_11: now also D12.2 (A)
- net X_12: now also D13.2 (A)
- net X_13: now also D14.2 (A)
- net X_14: now also D15.2 (A)
- net X_15: now also D16.2 (A)
- net X_2: now also D3.2 (A)
- net X_3: now also D4.2 (A)
- net X_4: now also D5.2 (A)
- net X_5: now also D6.2 (A)
- net X_6: now also D7.2 (A)
- net X_7: now also D8.2 (A)
- net X_8: now also D9.2 (A)
- net X_9: now also D10.2 (A)
- net Y_0: now also D17.2 (A)
- net Y_1: now also D18.2 (A)
- net Y_10: now also D27.2 (A)
- net Y_11: now also D28.2 (A)
- net Y_12: now also D29.2 (A)
- net Y_13: now also D30.2 (A)
- net Y_14: now also D31.2 (A)
- net Y_15: now also D32.2 (A)
- net Y_2: now also D19.2 (A)
- net Y_3: now also D20.2 (A)
- net Y_4: now also D21.2 (A)
- net Y_5: now also D22.2 (A)
- net Y_6: now also D23.2 (A)
- net Y_7: now also D24.2 (A)
- net Y_8: now also D25.2 (A)
- net Y_9: now also D26.2 (A)
- net ZR: now also D55.2 (A)
- net ZX: now also D49.2 (A)
- net ZY: now also D51.2 (A)
- new net: D1.1 (K), R1.2
- new net: D2.1 (K), R2.2
- new net: D3.1 (K), R3.2
- new net: D4.1 (K), R4.2
- new net: D5.1 (K), R5.2
- new net: D6.1 (K), R6.2
- new net: D7.1 (K), R7.2
- new net: D8.1 (K), R8.2
- new net: D9.1 (K), R9.2
- new net: D10.1 (K), R10.2
- new net: D11.1 (K), R11.2
- new net: D12.1 (K), R12.2
- new net: D13.1 (K), R13.2
- new net: D14.1 (K), R14.2
- new net: D15.1 (K), R15.2
- new net: D16.1 (K), R16.2
- new net: D17.1 (K), R17.2
- new net: D18.1 (K), R18.2
- new net: D19.1 (K), R19.2
- new net: D20.1 (K), R20.2
- new net: D21.1 (K), R21.2
- new net: D22.1 (K), R22.2
- new net: D23.1 (K), R23.2
- new net: D24.1 (K), R24.2
- new net: D25.1 (K), R25.2
- new net: D26.1 (K), R26.2
- new net: D27.1 (K), R27.2
- new net: D28.1 (K), R28.2
- new net: D29.1 (K), R29.2
- new net: D30.1 (K), R30.2
- new net: D31.1 (K), R31.2
- new net: D32.1 (K), R32.2
- new net: D33.1 (K), R33.2
- new net: D34.1 (K), R34.2
- new net: D35.1 (K), R35.2
- new net: D36.1 (K), R36.2
- new net: D37.1 (K), R37.2
- new net: D38.1 (K), R38.2
- new net: D39.1 (K), R39.2
- new net: D40.1 (K), R40.2
- new net: D41.1 (K), R41.2
- new net: D42.1 (K), R42.2
- new net: D43.1 (K), R43.2
- new net: D44.1 (K), R44.2
- new net: D45.1 (K), R45.2
- new net: D46.1 (K), R46.2
- new net: D47.1 (K), R47.2
- new net: D48.1 (K), R48.2
- new net: D49.1 (K), R49.2
- new net: D50.1 (K), R50.2
- new net: D51.1 (K), R51.2
- new net: D52.1 (K), R52.2
- new net: D53.1 (K), R53.2
- new net: D54.1 (K), R54.2
- new net: D55.1 (K), R55.2
- new net: D56.1 (K), R56.2
- new net +5V: J6.1
- new net GND: J6.2, R1.1, R10.1, R11.1, R12.1, R13.1, R14.1, R15.1, R16.1, R17.1, R18.1, R19.1, R2.1, R20.1, R21.1, R22.1, R23.1, R24.1, R25.1, R26.1, R27.1, R28.1, R29.1, R3.1, R30.1, R31.1, R32.1, R33.1, R34.1, R35.1, R36.1, R37.1, R38.1, R39.1, R4.1, R40.1, R41.1, R42.1, R43.1, R44.1, R45.1, R46.1, R47.1, R48.1, R49.1, R5.1, R50.1, R51.1, R52.1, R53.1, R54.1, R55.1, R56.1, R6.1, R7.1, R8.1, R9.1
Other:
- note added: "Control Input \nConnector"
- note added: "Output LEDs"
- note added: "Power Input"
- note removed: "Control Input Connector"
- moved on the sheet: J1, J2, J3, J4, J5
